File: I2CRJ45X8.sch (EAGLE design)
At the start: 59 parts, among them IC1 MCP23017SO, IC2 MCP23017SO, J1 M02X3-SHROUDED, J2 INT2A, J3 M02X3-PIN, J4 M02X3-PIN, J5 RJ45-X8, J6 M02X3-SHROUDED, J7 INT1A

Commit message: Converted to I2C-BREAKOUT header for v2.0 release
Parts:
- removed R41: 10K, SuperHouse-DiscreteSemi:RESISTOR0603
- removed SJ1: (no value), SuperHouse-Jumpers:SJ-NORMAL
- removed SJ2: SJC-NORMAL, SuperHouse-Jumpers:SJC-NORMAL
- J1, J6: value M02X3-SHROUDED -> I2C-BREAKOUT
- R40: value 10K -> 1K
Connections:
- removed net !RST: IC1.!RESET, IC2.!RESET, SJ1.1, SJ2.2
- removed net N$14: R41.1, SJ1.2
- net !RESET: now also IC1.!RESET, IC2.!RESET; no longer SJ2.1
- net VCC: no longer R41.2
Other:
- note added: "V2.0 (2020-04-06)"
- note removed: "V1.0 (2019-07-25)"
Changed lines of the file:
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@@
 <?xml version="1.0" encoding="utf-8"?>
 <!DOCTYPE eagle SYSTEM "eagle.dtd">
-<eagle version="9.5.0">
+<eagle version="9.6.0">
 <drawing>
 <settings>
@@
 <part name="LED2" library="SuperHouse-LEDs" library_urn="urn:adsk.eagle:library:11790571" deviceset="LED" device="0603" package3d_urn="urn:adsk.eagle:package:7066240/3" value="GREEN"/>
 <part name="R39" library="SuperHouse-DiscreteSemi" library_urn="urn:adsk.eagle:library:11768461" deviceset="RESISTOR" device="0603" package3d_urn="urn:adsk.eagle:package:11768543/2" value="10K"/>
-<part name="R40" library="SuperHouse-DiscreteSemi" library_urn="urn:adsk.eagle:library:11768461" deviceset="RESISTOR" device="0603" package3d_urn="urn:adsk.eagle:package:11768543/2" value="10K"/>
+<part name="R40" library="SuperHouse-DiscreteSemi" library_urn="urn:adsk.eagle:library:11768461" deviceset="RESISTOR" device="0603" package3d_urn="urn:adsk.eagle:package:11768543/2" value="1K"/>
 <part name="P+5" library="SuperHouse-SupplySymbols" library_urn="urn:adsk.eagle:library:11790503" deviceset="VCC" device=""/>
 <part name="GND6" library="SuperHouse-SupplySymbols" library_urn="urn:adsk.eagle:library:11790503" deviceset="GND" device=""/>
@@
 <part name="FID2" library="SuperHouse-Symbols" library_urn="urn:adsk.eagle:library:13228893" deviceset="FIDUCIAL" device="1X2.5" package3d_urn="urn:adsk.eagle:package:13228898/1"/>
 <part name="FID3" library="SuperHouse-Symbols" library_urn="urn:adsk.eagle:library:13228893" deviceset="FIDUCIAL" device="1X2.5" package3d_urn="urn:adsk.eagle:package:13228898/1"/>
-<part name="J6" library="SuperHouse-Connectors" library_urn="urn:adsk.eagle:library:11765989" deviceset="M02X3" device="-SHROUDED" package3d_urn="urn:adsk.eagle:package:13425426/3"/>
+<part name="J6" library="SuperHouse-Connectors" library_urn="urn:adsk.eagle:library:11765989" deviceset="M02X3" device="-SHROUDED" package3d_urn="urn:adsk.eagle:package:13425426/3" value="I2C-BREAKOUT"/>
 <part name="GND8" library="SuperHouse-SupplySymbols" library_urn="urn:adsk.eagle:library:11790503" deviceset="GND" device=""/>
 <part name="P+6" library="SuperHouse-SupplySymbols" library_urn="urn:adsk.eagle:library:11790503" deviceset="VCC" device=""/>
-<part name="J1" library="SuperHouse-Connectors" library_urn="urn:adsk.eagle:library:11765989" deviceset="M02X3" device="-SHROUDED" package3d_urn="urn:adsk.eagle:package:13425426/3"/>
+<part name="J1" library="SuperHouse-Connectors" library_urn="urn:adsk.eagle:library:11765989" deviceset="M02X3" device="-SHROUDED" package3d_urn="urn:adsk.eagle:package:13425426/3" value="I2C-BREAKOUT"/>
 <part name="GND4" library="SuperHouse-SupplySymbols" library_urn="urn:adsk.eagle:library:11790503" deviceset="GND" device=""/>
 <part name="P+4" library="SuperHouse-SupplySymbols" library_urn="urn:adsk.eagle:library:11790503" deviceset="VCC" device=""/>
 <part name="J2" library="SuperHouse-Connectors" library_urn="urn:adsk.eagle:library:11765989" deviceset="M01" device="-PLAIN" package3d_urn="urn:adsk.eagle:package:13097103/1" value="INT2A"/>
 <part name="J7" library="SuperHouse-Connectors" library_urn="urn:adsk.eagle:library:11765989" deviceset="M01" device="-PLAIN" package3d_urn="urn:adsk.eagle:package:13097103/1" value="INT1A"/>
-<part name="SJ1" library="SuperHouse-Jumpers" library_urn="urn:adsk.eagle:library:12190622" deviceset="SJ" device="-NORMAL" package3d_urn="urn:adsk.eagle:package:7066338/1"/>
-<part name="SJ2" library="SuperHouse-Jumpers" library_urn="urn:adsk.eagle:library:12190622" deviceset="SJC" device="-NORMAL" package3d_urn="urn:adsk.eagle:package:7066342/1"/>
-<part name="R41" library="SuperHouse-DiscreteSemi" library_urn="urn:adsk.eagle:library:11768461" deviceset="RESISTOR" device="0603" package3d_urn="urn:adsk.eagle:package:11768543/2" value="10K"/>
-<part name="P+3" library="SuperHouse-SupplySymbols" library_urn="urn:adsk.eagle:library:11790503" deviceset="VCC" device=""/>
 </parts>
 <sheets>
@@
 <frame x1="0" y1="0" x2="248.92" y2="185.42" columns="8" rows="5" layer="94"/>
 <text x="149.86" y="12.7" size="3.048" layer="94">8 Channel I2C RJ45 Breakout</text>
-<text x="215.9" y="6.858" size="1.778" layer="94">V1.0 (2019-07-25)</text>
+<text x="215.9" y="6.858" size="1.778" layer="94">V2.0 (2020-04-06)</text>
 <text x="149.606" y="6.858" size="1.778" layer="94">www.superhouse.tv/i2crj45x8</text>
 <text x="187.96" y="6.858" size="1.778" layer="94">SKU: I2CRJ45X8</text>
@@
 <attribute name="VALUE" x="35.56" y="139.7" size="1.778" layer="96" align="bottom-center"/>
 <attribute name="NAME" x="35.56" y="148.082" size="1.778" layer="95" align="bottom-center"/>
-</instance>
-<instance part="SJ1" gate="1" x="213.36" y="48.26" smashed="yes" rot="R90">
-<attribute name="NAME" x="210.82" y="45.72" size="1.778" layer="95" rot="R90"/>
-<attribute name="VALUE" x="217.17" y="45.72" size="1.778" layer="96" rot="R90"/>
-</instance>
-<instance part="SJ2" gate="G$1" x="213.36" y="38.1" smashed="yes" rot="R90">
-<attribute name="NAME" x="210.82" y="35.56" size="1.778" layer="95" rot="R90"/>
-</instance>
-<instance part="R41" gate="G$1" x="213.36" y="58.42" smashed="yes" rot="MR90">
-<attribute name="NAME" x="214.8586" y="54.61" size="1.778" layer="95" rot="MR90"/>
-<attribute name="VALUE" x="215.138" y="59.69" size="1.778" layer="96" rot="MR90"/>
-</instance>
-<instance part="P+3" gate="1" x="213.36" y="66.04" smashed="yes">
-<attribute name="VALUE" x="212.344" y="69.596" size="1.778" layer="96"/>
 </instance>
 </instances>
@@
 <wire x1="160.02" y1="35.56" x2="160.02" y2="43.18" width="0.1524" layer="91"/>
 </segment>
-<segment>
-<pinref part="R41" gate="G$1" pin="2"/>
-<pinref part="P+3" gate="1" pin="VCC"/>
-<wire x1="213.36" y1="63.5" x2="213.36" y2="66.04" width="0.1524" layer="91"/>
-</segment>
 </net>
 <net name="N$2" class="0">
@@
 </segment>
 <segment>
-<pinref part="SJ2" gate="G$1" pin="1"/>
-<wire x1="213.36" y1="33.02" x2="213.36" y2="30.48" width="0.1524" layer="91"/>
-<wire x1="213.36" y1="30.48" x2="208.28" y2="30.48" width="0.1524" layer="91"/>
-<label x="208.28" y="30.48" size="1.27" layer="95" rot="R180" xref="yes"/>
-</segment>
-</net>
-<net name="N$9" class="0">
-<segment>
-<pinref part="IC2" gate="G$1" pin="INTA"/>
-<wire x1="167.64" y1="144.78" x2="165.1" y2="144.78" width="0.1524" layer="91"/>
-<pinref part="J2" gate="G$1" pin="1"/>
-</segment>
-</net>
-<net name="N$10" class="0">
-<segment>
-<pinref part="IC1" gate="G$1" pin="INTA"/>
-<pinref part="J7" gate="G$1" pin="1"/>
-<wire x1="43.18" y1="144.78" x2="45.72" y2="144.78" width="0.1524" layer="91"/>
-</segment>
-</net>
-<net name="!RST" class="0">
-<segment>
-<pinref part="SJ1" gate="1" pin="1"/>
-<pinref part="SJ2" gate="G$1" pin="2"/>
-<wire x1="213.36" y1="43.18" x2="208.28" y2="43.18" width="0.1524" layer="91"/>
-<junction x="213.36" y="43.18"/>
-<label x="208.28" y="43.18" size="1.27" layer="95" rot="R180" xref="yes"/>
-</segment>
-<segment>
 <pinref part="IC1" gate="G$1" pin="!RESET"/>
 <wire x1="45.72" y1="149.86" x2="40.64" y2="149.86" width="0.1524" layer="91"/>
@@
 </segment>
 </net>
-<net name="N$14" class="0">
-<segment>
-<pinref part="R41" gate="G$1" pin="1"/>
-<pinref part="SJ1" gate="1" pin="2"/>
-</segment>
-</net>
+<net name="N$9" class="0">
+<segment>
+<pinref part="IC2" gate="G$1" pin="INTA"/>
+<wire x1="167.64" y1="144.78" x2="165.1" y2="144.78" width="0.1524" layer="91"/>
+<pinref part="J2" gate="G$1" pin="1"/>
+</segment>
+</net>
+<net name="N$10" class="0">
+<segment>
+<pinref part="IC1" gate="G$1" pin="INTA"/>
+<pinref part="J7" gate="G$1" pin="1"/>
+<wire x1="43.18" y1="144.78" x2="45.72" y2="144.78" width="0.1524" layer="91"/>
+</segment>
+</net>
