File: Hardware/I2CRJ45X8.sch (EAGLE design)
At the start: 91 parts, among them IC1 MCP23017SO, IC2 MCP23017SO, IC3 MCP23017SO, IC4 MCP23017SO, J1 I2C-BREAKOUT, J2 I2C-BREAKOUT, J3 M01-PLAIN, J4 RJ45-X8, J5 RJ45-X8

Commit message: Major update based on 24-port project. Use solder jumpers for I2C address selection.
Parts:
- removed C3, C4: 10uF, SuperHouse-DiscreteSemi:CAP0805
- removed C5: 330uF 50V, SuperHouse-DiscreteSemi:CAP_POLG
- removed IC3, IC4: MCP23017SO, SuperHouse-ICs:MCP23017SO
- removed J5: RJ45-X8, SuperHouse-Connectors:RJ45-X8
- removed R44, R45, R46, R47, R48, R49, R50, R51, R52, R53, R54, R55, R56, R57, R58, R59, R60, R61, R62, R63, R64: 1K, SuperHouse-DiscreteSemi:RESISTOR0603
- removed R65, R66, R67, R68: 4K7, SuperHouse-DiscreteSemi:RESISTOR0603
- removed R69: 22K, SuperHouse-DiscreteSemi:RESISTOR0603
- added SJ4, SJ7: A0, SuperHouse-Jumpers:SJ-NORMAL
- added SJ5, SJ8: A1, SuperHouse-Jumpers:SJ-NORMAL
- added SJ6, SJ9: A2, SuperHouse-Jumpers:SJ-NORMAL
- R33, R34, R35, R36: value 1K -> 4K7
- R37, R38, R39, R40, R41, R42, R43: value 1K -> 10K
- SJ3: device SuperHouse-Jumpers:SJC-NORMAL -> SuperHouse-Jumpers:SJ-NORMAL
Connections:
- removed net 2A1: J5.A1, R33.2
- removed net 2A2: J5.A2, R35.2
- removed net 2A3: J5.A3, R34.2
- removed net 2A6: J5.A6, R36.2
- removed net 2B1: J5.B1, R49.2
- removed net 2B2: J5.B2, R47.2
- removed net 2B3: J5.B3, R45.2
- removed net 2B6: J5.B6, R43.2
- removed net 2C1: J5.C1, R51.2
- removed net 2C2: J5.C2, R53.2
- removed net 2C3: J5.C3, R52.2
- removed net 2C6: J5.C6, R54.2
- removed net 2D1: J5.D1, R40.2
- removed net 2D2: J5.D2, R63.2
- removed net 2D3: J5.D3, R61.2
- removed net 2D6: J5.D6, R59.2
- removed net 2E1: J5.E1, R41.2
- removed net 2E2: J5.E2, R38.2
- removed net 2E3: J5.E3, R37.2
- removed net 2E6: J5.E6, R42.2
- removed net 2F1: J5.F1, R50.2
- removed net 2F2: J5.F2, R48.2
- removed net 2F3: J5.F3, R46.2
- removed net 2F6: J5.F6, R44.2
- removed net 2G1: J5.G1, R57.2
- removed net 2G2: J5.G2, R56.2
- removed net 2G3: J5.G3, R55.2
- removed net 2G6: J5.G6, R58.2
- removed net 2H1: J5.H1, R39.2
- removed net 2H2: J5.H2, R64.2
- removed net 2H3: J5.H3, R62.2
- removed net 2H6: J5.H6, R60.2
- removed net GPA0-3: IC3.GPA0, R33.1
- removed net GPA0-4: IC4.GPA0, R51.1
- removed net GPA1-3: IC3.GPA1, R35.1
- removed net GPA1-4: IC4.GPA1, R53.1
- removed net GPA2-3: IC3.GPA2, R34.1
- removed net GPA2-4: IC4.GPA2, R52.1
- removed net GPA3-3: IC3.GPA3, R36.1
- removed net GPA3-4: IC4.GPA3, R54.1
- removed net GPA4-3: IC3.GPA4, R41.1
- removed net GPA4-4: IC4.GPA4, R57.1
- removed net GPA5-3: IC3.GPA5, R38.1
- removed net GPA5-4: IC4.GPA5, R56.1
- removed net GPA6-3: IC3.GPA6, R37.1
- removed net GPA6-4: IC4.GPA6, R55.1
- removed net GPA7-3: IC3.GPA7, R42.1
- removed net GPA7-4: IC4.GPA7, R58.1
- removed net GPB0-3: IC3.GPB0, R49.1
- removed net GPB0-4: IC4.GPB0, R40.1
- removed net GPB1-3: IC3.GPB1, R47.1
- removed net GPB1-4: IC4.GPB1, R63.1
- removed net GPB2-3: IC3.GPB2, R45.1
- removed net GPB2-4: IC4.GPB2, R61.1
- removed net GPB3-3: IC3.GPB3, R43.1
- removed net GPB3-4: IC4.GPB3, R59.1
- removed net GPB4-3: IC3.GPB4, R50.1
- removed net GPB4-4: IC4.GPB4, R39.1
- removed net GPB5-3: IC3.GPB5, R48.1
- removed net GPB5-4: IC4.GPB5, R64.1
- removed net GPB6-3: IC3.GPB6, R46.1
- removed net GPB6-4: IC4.GPB6, R62.1
- removed net GPB7-3: IC3.GPB7, R44.1
- removed net GPB7-4: IC4.GPB7, R60.1
- new net N$10: IC2.A1, R37.2, SJ8.1
- new net N$11: IC2.A0, R43.2, SJ7.1
- new net N$4: IC1.A2, R42.2, SJ6.1
- new net N$5: IC1.A1, R41.2, SJ5.1
- new net N$6: IC1.A0, R40.2, SJ4.1
- new net N$9: IC2.A2, R38.2, SJ9.1
- net !INT: no longer IC3.INTA, IC4.INTA
- net !RESET: now also R39.1; no longer IC3.!RESET, IC4.!RESET, R69.1
- net GND: now also R37.1, R38.1, R40.1, R41.1, R42.1, R43.1; no longer C3.2, C4.2, C5.-, IC1.A0, IC1.A1, IC1.A2, IC2.A1, IC2.A2, IC3.A0, IC3.A2, IC3.VSS, IC4.A2, IC4.VSS, J5.A7, J5.A8, J5.B7, J5.B8, J5.C7, J5.C8, J5.D7, J5.D8, J5.E7, J5.E8, J5.F7, J5.F8, J5.G7, J5.G8, J5.GND0, J5.GND1, J5.GND2, J5.GND3, J5.GND4, J5.GND5, J5.H7, J5.H8
- net N$1: now also R35.2; no longer R67.2
- net N$2: now also R36.2; no longer R68.2
- net N$3: now also R39.2; no longer R69.2
- net N$7: now also R33.1; no longer R65.1
- net N$8: now also R34.1; no longer R66.1
- net SCL: now also R35.1; no longer IC3.SCL, IC4.SCL, R67.1
- net SDA: now also R36.1; no longer IC3.SDA, IC4.SDA, R68.1
- net VCC: now also R33.2, SJ4.2, SJ5.2, SJ6.2, SJ7.2, SJ8.2, SJ9.2; no longer C3.1, C4.1, IC2.A0, IC3.A1, IC3.VDD, IC4.A0, IC4.A1, IC4.VDD, R65.2
- net VIN: now also R34.2; no longer C5.+, J5.A4, J5.A5, J5.B4, J5.B5, J5.C4, J5.C5, J5.D4, J5.D5, J5.E4, J5.E5, J5.F4, J5.F5, J5.G4, J5.G5, J5.H4, J5.H5, R66.2
Other:
- note added: "8-Port I2C RJ45 Breakout"
- note added: "I2C pullups are disabled by default. Solder bridge across SJ1 and SJ2 to enable. Reset pullup is disabled by default. Solder bridge across SJ3 to enable."
- note added: "SKU: I2CRJ45X8"
- note added: "www.superhouse.tv/i2crj45x8"
- note removed: "16-Channel I2C RJ45 Breakout"
- note removed: "I2C Addr: 0x21"
- note removed: "I2C Addr: 0x22"
- note removed: "I2C Addr: 0x23"
- note removed: "I2C pullups are disabled by default. Solder bridge across SJ2 and SJ3 to enable. Reset pullup is enabled by default. Cut track between pads to disable."
- note removed: "SKU: I2CRJ45X16"
- note removed: "www.superhouse.tv/i2crj45x16"
