File: Hardware/I2CRJ45X8-old.brd (EAGLE design)
At the start: 76 x 50 mm, 60 parts, among them IC1 MCP23017SO, IC2 MCP23017SO, J1 I2C-BREAKOUT, J2 INT2A, J3 M02X3-PIN, J4 M02X3-PIN, J5 RJ45-X8, J6 I2C-BREAKOUT, J7 INT1A

Commit message: Moved in files from x16 version to begin conversion.
Parts:
- R33: value 1K -> 4K7
- R39: value 10K -> 4K7
Changed lines of the file:
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@@
 <attribute name="VALUE" x="73.0348" y="19.016" size="0.4064" layer="27" rot="R270"/>
 </element>
-<element name="R39" library="SuperHouse-DiscreteSemi" library_urn="urn:adsk.eagle:library:11768461" package="R0603" package3d_urn="urn:adsk.eagle:package:11768543/2" value="10K" x="71" y="22" smashed="yes" rot="R90">
+<element name="R39" library="SuperHouse-DiscreteSemi" library_urn="urn:adsk.eagle:library:11768461" package="R0603" package3d_urn="urn:adsk.eagle:package:11768543/2" value="4K7" x="71" y="22" smashed="yes" rot="R90">
 <attribute name="NAME" x="70.492" y="21.111" size="0.4064" layer="25" font="vector" rot="R90"/>
 <attribute name="VALUE" x="71.9652" y="20.984" size="0.4064" layer="27" font="vector" rot="R90"/>
 </element>
-<element name="R33" library="SuperHouse-DiscreteSemi" library_urn="urn:adsk.eagle:library:11768461" package="R0603" package3d_urn="urn:adsk.eagle:package:11768543/2" value="1K" x="74" y="22" smashed="yes" rot="R90">
+<element name="R33" library="SuperHouse-DiscreteSemi" library_urn="urn:adsk.eagle:library:11768461" package="R0603" package3d_urn="urn:adsk.eagle:package:11768543/2" value="4K7" x="74" y="22" smashed="yes" rot="R90">
 <attribute name="NAME" x="73.492" y="21.111" size="0.4064" layer="25" font="vector" rot="R90"/>
 <attribute name="VALUE" x="74.9652" y="20.984" size="0.4064" layer="27" font="vector" rot="R90"/>
